File: DROID.brd (EAGLE design)
At the start: 160 x 100 mm, 92 parts

Commit message: getti'n close
Connections:
- removed net Q13_E: Q13.2
- removed net Q14_E: Q14.2
- removed net Q6_C: Q6.3
- removed net Q6_E: Q6.2
- removed net R22_A: R18.1, R22.1
- removed net R27_A: R27.1
- removed net R29_A: R23.1, R29.1
- removed net R49_A: R49.1
- removed net R51_A: R51.1
- removed net R52_A: R52.1
- removed net R68_A: R68.1
- removed net R68_B: R68.2
- removed net R6_A: R6.1
- removed net R6_B: R6.2
- removed net R71_B: R71.2
- removed net R7_A: R7.1
- removed net R7_B: R7.2
- removed net VCC_5V: JP14.5, U$5.2, U$5.23, U$5.32, U$5.4, U$5.7
- net HE_5V: now also Q6.3
- net H_L: now also R52.1
- net H_MID: now also R49.1
- net H_R: now also R51.1
- net L_ID: now also R18.1, R22.1
- net L_LED: now also R6.1
- net P0.14: now also R68.2, R71.2; no longer U$5.18
- net P0.15: now also U$5.18; no longer U$5.19
- net Q12_B: now also R68.1
- net Q13_C: now also R6.2
- net Q14_C: now also R7.1
- net Q6_B: now also R27.1
- net R_ID: now also R23.1, R29.1
- net R_LED: now also R7.2
- net SWCLK: now also U$5.19
- net U7_VOUT: now also Q13.2, Q14.2, Q6.2
- net VCC_33: now also JP14.5, U$5.2, U$5.23, U$5.32, U$5.4, U$5.7
Changed lines of the file:
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@@
 <signal name="Q14_C">
 <contactref element="Q14" pad="3"/>
-</signal>
-<signal name="Q14_E">
-<contactref element="Q14" pad="2"/>
-</signal>
-<signal name="R51_A">
-<contactref element="R51" pad="1"/>
+<contactref element="R7" pad="1"/>
+<wire x1="-29.21" y1="12.43" x2="-44.03" y2="15.24" width="0" layer="19" extent="1-1"/>
 </signal>
 <signal name="R51_B">
@@
 <wire x1="-16.93" y1="21.59" x2="-44.29" y2="-7.7" width="0" layer="19" extent="1-1"/>
 </signal>
-<signal name="R52_A">
-<contactref element="R52" pad="1"/>
-</signal>
 <signal name="R52_B">
 <contactref element="R52" pad="2"/>
@@
 <wire x1="-42.33" y1="19.05" x2="-31.67" y2="-17.62" width="0" layer="19" extent="1-1"/>
 </signal>
-<signal name="R49_A">
-<contactref element="R49" pad="1"/>
-</signal>
 <signal name="R49_B">
 <contactref element="R49" pad="2"/>
@@
 <wire x1="-23.28" y1="19.05" x2="-38.72" y2="-20.32" width="0" layer="19" extent="1-1"/>
 </signal>
-<signal name="R27_A">
-<contactref element="R27" pad="1"/>
-</signal>
 <signal name="R27_B">
 <contactref element="R27" pad="2"/>
@@
 <wire x1="-16.93" y1="19.05" x2="-33.72" y2="-20.32" width="0" layer="19" extent="1-1"/>
 </signal>
-<signal name="R7_A">
-<contactref element="R7" pad="1"/>
-</signal>
-<signal name="R7_B">
-<contactref element="R7" pad="2"/>
-</signal>
-<signal name="R6_A">
-<contactref element="R6" pad="1"/>
-</signal>
-<signal name="R6_B">
-<contactref element="R6" pad="2"/>
-</signal>
 <signal name="R54_A">
 <contactref element="R54" pad="1"/>
@@
 <signal name="Q6_B">
 <contactref element="Q6" pad="1"/>
-</signal>
-<signal name="Q6_C">
-<contactref element="Q6" pad="3"/>
-</signal>
-<signal name="Q6_E">
-<contactref element="Q6" pad="2"/>
+<contactref element="R27" pad="1"/>
+<wire x1="-18.63" y1="19.05" x2="-36.51" y2="10.43" width="0" layer="19" extent="1-1"/>
 </signal>
 <signal name="Q13_B">
@@
 <signal name="Q13_C">
 <contactref element="Q13" pad="3"/>
-</signal>
-<signal name="Q13_E">
-<contactref element="Q13" pad="2"/>
+<contactref element="R6" pad="2"/>
+<wire x1="-22.86" y1="12.43" x2="-35.98" y2="15.24" width="0" layer="19" extent="1-1"/>
 </signal>
 <signal name="Q10_B">
@@
 <wire x1="-23.28" y1="26.67" x2="-29.63" y2="26.67" width="0" layer="19" extent="1-1"/>
 </signal>
-<signal name="R29_A">
-<contactref element="R29" pad="1"/>
-<contactref element="R23" pad="1"/>
-<wire x1="-24.98" y1="26.67" x2="-18.63" y2="26.67" width="0" layer="19" extent="1-1"/>
-</signal>
 <signal name="R29_B">
 <contactref element="R29" pad="2"/>
@@
 <wire x1="-16.93" y1="26.67" x2="-35.48" y2="-17.62" width="0" layer="19" extent="1-1"/>
 </signal>
-<signal name="R22_A">
-<contactref element="R22" pad="1"/>
-<contactref element="R18" pad="1"/>
-<wire x1="-31.33" y1="26.67" x2="-37.68" y2="26.67" width="0" layer="19" extent="1-1"/>
-</signal>
 <signal name="R22_B">
 <contactref element="R22" pad="2"/>
@@
 <contactref element="C20A" pad="2"/>
 </signal>
-<signal name="R68_A">
-<contactref element="R68" pad="1"/>
-</signal>
-<signal name="R68_B">
-<contactref element="R68" pad="2"/>
-</signal>
 <signal name="R26_A">
 <contactref element="R26" pad="1"/>
@@
 <signal name="R26_B">
 <contactref element="R26" pad="2"/>
-</signal>
-<signal name="R71_B">
-<contactref element="R71" pad="2"/>
 </signal>
 <signal name="R25_B">
@@
 <signal name="Q12_B">
 <contactref element="Q12" pad="1"/>
+<contactref element="R68" pad="1"/>
+<wire x1="-37.68" y1="21.59" x2="-37.78" y2="1.54" width="0" layer="19" extent="1-1"/>
 </signal>
 <signal name="Q12_C">
@@
 <signal name="P0.14">
 <contactref element="U$4" pad="P$25"/>
-<contactref element="U$5" pad="18"/>
-<wire x1="-24.29" y1="-13.89" x2="-41.72" y2="-38.32" width="0" layer="19" extent="1-1"/>
+<contactref element="R68" pad="2"/>
+<contactref element="R71" pad="2"/>
+<wire x1="-29.63" y1="21.59" x2="-24.29" y2="-13.89" width="0" layer="19" extent="1-1"/>
+<wire x1="-35.98" y1="21.59" x2="-29.63" y2="21.59" width="0" layer="19" extent="1-1"/>
 </signal>
 <signal name="P0.15">
 <contactref element="U$4" pad="P$26"/>
-<contactref element="U$5" pad="19"/>
-<wire x1="-24.29" y1="-12.62" x2="-40.72" y2="-38.32" width="0" layer="19" extent="1-1"/>
+<contactref element="U$5" pad="18"/>
+<wire x1="-24.29" y1="-12.62" x2="-41.72" y2="-38.32" width="0" layer="19" extent="1-1"/>
 </signal>
 <signal name="P0.17">
@@
 <contactref element="JP14" pad="1"/>
 <wire x1="-25.72" y1="-20.32" x2="-82.55" y2="-78.74" width="0" layer="19" extent="1-1"/>
-</signal>
-<signal name="VCC_5V">
-<contactref element="U$5" pad="2"/>
-<contactref element="U$5" pad="4"/>
-<contactref element="U$5" pad="7"/>
-<contactref element="U$5" pad="23"/>
-<contactref element="U$5" pad="32"/>
-<contactref element="JP14" pad="5"/>
-<wire x1="-36.72" y1="-38.32" x2="-72.39" y2="-78.74" width="0" layer="19" extent="1-1"/>
-<wire x1="-27.72" y1="-38.32" x2="-36.72" y2="-38.32" width="0" layer="19" extent="1-1"/>
-<wire x1="-28.72" y1="-20.32" x2="-27.72" y2="-38.32" width="0" layer="19" extent="1-1"/>
-<wire x1="-26.72" y1="-20.32" x2="-28.72" y2="-20.32" width="0" layer="19" extent="1-1"/>
-<wire x1="-31.72" y1="-20.32" x2="-28.72" y2="-20.32" width="0" layer="19" extent="1-1"/>
 </signal>
 <signal name="GND">
@@
 <signal name="HE_5V">
 <contactref element="JP13" pad="5"/>
+<contactref element="Q6" pad="3"/>
+<wire x1="-35.56" y1="12.43" x2="-72.39" y2="-73.66" width="0" layer="19" extent="1-1"/>
 </signal>
 <signal name="H_R">
 <contactref element="JP10" pad="1"/>
+<contactref element="R51" pad="1"/>
+<wire x1="-18.63" y1="21.59" x2="-82.55" y2="-58.42" width="0" layer="19" extent="1-1"/>
 </signal>
 <signal name="H_L">
 <contactref element="JP10" pad="2"/>
+<contactref element="R52" pad="1"/>
+<wire x1="-44.03" y1="19.05" x2="-80.01" y2="-58.42" width="0" layer="19" extent="1-1"/>
 </signal>
 <signal name="H_MID">
 <contactref element="JP10" pad="3"/>
+<contactref element="R49" pad="1"/>
+<wire x1="-37.68" y1="19.05" x2="-77.47" y2="-58.42" width="0" layer="19" extent="1-1"/>
 </signal>
 <signal name="VCC_ON">
@@
 <signal name="L_ID">
 <contactref element="JP8" pad="1"/>
+<contactref element="R22" pad="1"/>
+<contactref element="R18" pad="1"/>
+<wire x1="-37.68" y1="26.67" x2="-82.55" y2="-48.26" width="0" layer="19" extent="1-1"/>
+<wire x1="-31.33" y1="26.67" x2="-37.68" y2="26.67" width="0" layer="19" extent="1-1"/>
 </signal>
 <signal name="L_LED">
 <contactref element="JP8" pad="3"/>
+<contactref element="R6" pad="1"/>
+<wire x1="-37.68" y1="15.24" x2="-77.47" y2="-48.26" width="0" layer="19" extent="1-1"/>
 </signal>
 <signal name="R_ID">
 <contactref element="JP7" pad="1"/>
+<contactref element="R29" pad="1"/>
+<contactref element="R23" pad="1"/>
+<wire x1="-24.98" y1="26.67" x2="-82.55" y2="-43.18" width="0" layer="19" extent="1-1"/>
+<wire x1="-18.63" y1="26.67" x2="-24.98" y2="26.67" width="0" layer="19" extent="1-1"/>
 </signal>
 <signal name="R_LED">
 <contactref element="JP7" pad="3"/>
+<contactref element="R7" pad="2"/>
+<wire x1="-42.33" y1="15.24" x2="-77.47" y2="-43.18" width="0" layer="19" extent="1-1"/>
 </signal>
 <signal name="HED_DET">
@@
 <contactref element="R76" pad="2"/>
 <contactref element="C31" pad="2"/>
-<wire x1="-74.93" y1="-68.58" x2="-82.55" y2="-83.82" width="0" layer="19" extent="1-1"/>
-<wire x1="-44.29" y1="-15.32" x2="-74.93" y2="-68.58" width="0" layer="19" extent="1-1"/>
-<wire x1="-16.93" y1="24.13" x2="-44.29" y2="-15.32" width="0" layer="19" extent="1-1"/>
+<contactref element="U$5" pad="2"/>
+<contactref element="U$5" pad="4"/>
+<contactref element="U$5" pad="7"/>
+<contactref element="U$5" pad="23"/>
+<contactref element="U$5" pad="32"/>
+<contactref element="JP14" pad="5"/>
+<wire x1="-72.39" y1="-78.74" x2="-82.55" y2="-83.82" width="0" layer="19" extent="1-1"/>
+<wire x1="-74.93" y1="-68.58" x2="-72.39" y2="-78.74" width="0" layer="19" extent="1-1"/>
+<wire x1="-36.72" y1="-38.32" x2="-74.93" y2="-68.58" width="0" layer="19" extent="1-1"/>
+<wire x1="-27.72" y1="-38.32" x2="-36.72" y2="-38.32" width="0" layer="19" extent="1-1"/>
+<wire x1="-28.72" y1="-20.32" x2="-27.72" y2="-38.32" width="0" layer="19" extent="1-1"/>
+<wire x1="-26.72" y1="-20.32" x2="-28.72" y2="-20.32" width="0" layer="19" extent="1-1"/>
+<wire x1="-31.72" y1="-20.32" x2="-28.72" y2="-20.32" width="0" layer="19" extent="1-1"/>
+<wire x1="-44.29" y1="-15.32" x2="-31.72" y2="-20.32" width="0" layer="19" extent="1-1"/>
+<wire x1="-16.93" y1="24.13" x2="-26.72" y2="-20.32" width="0" layer="19" extent="1-1"/>
 <wire x1="-16.93" y1="39.37" x2="-16.93" y2="24.13" width="0" layer="19" extent="1-1"/>
 </signal>
@@
 <contactref element="JP12" pad="2"/>
 <contactref element="U$4" pad="P$27"/>
-<wire x1="-24.29" y1="-11.35" x2="-80.01" y2="-68.58" width="0" layer="19" extent="1-1"/>
+<contactref element="U$5" pad="19"/>
+<wire x1="-40.72" y1="-38.32" x2="-80.01" y2="-68.58" width="0" layer="19" extent="1-1"/>
+<wire x1="-24.29" y1="-11.35" x2="-40.72" y2="-38.32" width="0" layer="19" extent="1-1"/>
 </signal>
 <signal name="HEAD_OUT_A">
@@
 <contactref element="L9" pad="2"/>
 <contactref element="Q10" pad="2"/>
+<contactref element="Q6" pad="2"/>
+<contactref element="Q14" pad="2"/>
+<contactref element="Q13" pad="2"/>
 <wire x1="-81.6" y1="-86.36" x2="-107.95" y2="-93.04" width="0" layer="19" extent="1-1"/>
-<wire x1="-15.56" y1="10.43" x2="-81.6" y2="-86.36" width="0" layer="19" extent="1-1"/>
+<wire x1="-34.61" y1="10.43" x2="-81.6" y2="-86.36" width="0" layer="19" extent="1-1"/>
+<wire x1="-28.26" y1="10.43" x2="-34.61" y2="10.43" width="0" layer="19" extent="1-1"/>
+<wire x1="-21.91" y1="10.43" x2="-28.26" y2="10.43" width="0" layer="19" extent="1-1"/>
+<wire x1="-15.56" y1="10.43" x2="-21.91" y2="10.43" width="0" layer="19" extent="1-1"/>
 <wire x1="-16.93" y1="34.29" x2="-15.56" y2="10.43" width="0" layer="19" extent="1-1"/>
 </signal>

Commit message: done for now
Connections:
- removed net C19_B: C19.2
- removed net C21_B: C21.2
- removed net C23_A: C23.1
- removed net C23_B: C23.2
- removed net C24_A: C24.1
- removed net C24_B: C24.2
- removed net C25_A: C25.1
- removed net C25_B: C25.2
- removed net C29_A: C29.1
- removed net C29_B: C29.2
- removed net C38_B: C38.2
- removed net C39_A: C39.1
- removed net C39_B: C39.2
- removed net F1_1: F1.P$1
- removed net F1_2: F1.P$2
- removed net L11_1: L11.1
- removed net L11_2: L11.2
- removed net L12_1: L12.1
- removed net L12_2: L12.2
- removed net L13_1: L13.1
- removed net L13_2: L13.2
- removed net L14_1: L14.1
- removed net L14_2: L14.2
- removed net N$113: C22A.1
- removed net N$114: C22A.2
- removed net N$94: C20A.2
- removed net R26_B: R26.2
- removed net R30_A: R30.1
- removed net R30_B: R30.2
- removed net R54_A: R54.1
- removed net R54_B: R54.2
- removed net R77_A: R77.1
- removed net U7_VOUT: C33.2, L9.2, Q10.2, Q13.2, Q14.2, Q6.2, U7.2, U7.2@1
- new net GND_INDUCTED: L14.2, U7.3
- new net SP+_OUT: C38.2, JP6.1, L12.1
- new net SP-_OUT: C39.2, JP6.2, L11.1
- net BAT+: now also F1.P$2
- net GND: now also C22A.1, C23.1, C24.1, C25.1, C29.1, C39.1, L14.1; no longer U7.3
- net Q10_B: now also R54.2
- net Q12_C: now also C29.2
- net R26_A: now also C21.2
- net SP+: now also L12.2; no longer JP6.1
- net SP-: now also L11.2; no longer JP6.2
- net U7_VIN: now also L13.2, Q10.2, R54.1
- net U8_VOUT: now also C24.2, C25.2, R77.1
- net VCC_33: now also C20A.2, C22A.2, C23.2, C33.2, L9.2, Q13.2, Q14.2, Q6.2, R26.2, R30.1, R30.2, U7.2, U7.2@1
- net VCC_ON: now also L13.1
- net VCV_M: now also C19.2, F1.P$1
