File: DROID.brd (EAGLE design)
At the start: 160 x 100 mm, 92 parts

Commit message: saving before cleanup
Connections:
- removed net C16_B: C16.2
- removed net C17_B: C17.2
- removed net C18_B: C18.2
- removed net C27_B: C27.2
- removed net C28_B: C28.2
- removed net D14_A: D14.A
- removed net N$135: U$3.4
- removed net N$137: U$3.2
- removed net N$138: U$3.8
- removed net N$143: U$2.4
- removed net N$145: U$2.2
- removed net N$146: U$2.8
- removed net N$151: U$1.4
- removed net N$153: U$1.2
- removed net N$154: U$1.8
- removed net N$16: R47_OR_42.2
- removed net R43_B: R43.2
- removed net R44_B: R44.2
- removed net R45_B: R45.2
- net HEAD_IN_A: now also R43.2
- net HEAD_IN_B: now also R45.2
- net LEFT_IN_A: now also R44.2
- net LEFT_IN_B: now also R47_OR_42.2
- net R62_B: no longer R62.2
- net R63_B: no longer R63.2
- net RIGHT_IN_A: now also R62.2
- net RIGHT_IN_B: now also R63.2
- net SWDIO: now also D14.A
- net VCV_M: now also C16.2, C17.2, C18.2, C27.2, C28.2, U$1.4, U$2.4, U$3.4
Changed lines of the file:
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@@
 </elements>
 <signals>
-<signal name="C27_B">
-<contactref element="C27" pad="2"/>
-</signal>
-<signal name="C18_B">
-<contactref element="C18" pad="2"/>
-</signal>
-<signal name="C28_B">
-<contactref element="C28" pad="2"/>
-</signal>
 <signal name="R62_B">
-<contactref element="R62" pad="2"/>
 <contactref element="U$4" pad="P$19"/>
-<wire x1="-43.6" y1="29.21" x2="-30.4" y2="-17.62" width="0" layer="19" extent="1-1"/>
-</signal>
-<signal name="R44_B">
-<contactref element="R44" pad="2"/>
 </signal>
 <signal name="R63_B">
-<contactref element="R63" pad="2"/>
 <contactref element="U$4" pad="P$20"/>
-<wire x1="-38.52" y1="29.21" x2="-29.13" y2="-17.62" width="0" layer="19" extent="1-1"/>
-</signal>
-<signal name="N$16">
-<contactref element="R47_OR_42" pad="2"/>
 </signal>
 <signal name="Q14_B">
@@
 <wire x1="-42.33" y1="34.29" x2="-36.83" y2="3.54" width="0" layer="19" extent="1-1"/>
 </signal>
-<signal name="C16_B">
-<contactref element="C16" pad="2"/>
-</signal>
-<signal name="C17_B">
-<contactref element="C17" pad="2"/>
-</signal>
-<signal name="R43_B">
-<contactref element="R43" pad="2"/>
-</signal>
-<signal name="R45_B">
-<contactref element="R45" pad="2"/>
-</signal>
 <signal name="HEAD_OUT_B">
 <contactref element="U$3" pad="5"/>
@@
 </signal>
 <signal name="HEAD_IN_B">
+<contactref element="U$4" pad="P$4"/>
+<contactref element="R45" pad="2"/>
 <contactref element="U$3" pad="3"/>
-<contactref element="U$4" pad="P$4"/>
 <wire x1="-24.765" y1="1.765" x2="-44.29" y2="-10.24" width="0" layer="19" extent="1-1"/>
+<wire x1="-15.66" y1="31.75" x2="-24.765" y2="1.765" width="0" layer="19" extent="1-1"/>
 </signal>
 <signal name="HEAD_IN_A">
+<contactref element="U$4" pad="P$3"/>
+<contactref element="R43" pad="2"/>
 <contactref element="U$3" pad="1"/>
-<contactref element="U$4" pad="P$3"/>
 <wire x1="-27.305" y1="1.765" x2="-44.29" y2="-8.97" width="0" layer="19" extent="1-1"/>
-</signal>
-<signal name="N$135">
-<contactref element="U$3" pad="4"/>
-</signal>
-<signal name="N$137">
-<contactref element="U$3" pad="2"/>
-</signal>
-<signal name="N$138">
-<contactref element="U$3" pad="8"/>
+<wire x1="-20.74" y1="31.75" x2="-27.305" y2="1.765" width="0" layer="19" extent="1-1"/>
 </signal>
 <signal name="RIGHT_OUT_B">
@@
 <wire x1="-20.955" y1="8.395" x2="-69.85" y2="-34.29" width="0" layer="19" extent="1-1"/>
 </signal>
-<signal name="RIGHT_IN_B">
-<contactref element="U$2" pad="3"/>
-</signal>
-<signal name="RIGHT_IN_A">
-<contactref element="U$2" pad="1"/>
-</signal>
-<signal name="N$143">
-<contactref element="U$2" pad="4"/>
-</signal>
-<signal name="N$145">
-<contactref element="U$2" pad="2"/>
-</signal>
-<signal name="N$146">
-<contactref element="U$2" pad="8"/>
-</signal>
 <signal name="LEFT_OUT_B">
 <contactref element="U$1" pad="5"/>
@@
 <contactref element="U$1" pad="3"/>
 <contactref element="U$4" pad="P$10"/>
+<contactref element="R47_OR_42" pad="2"/>
 <wire x1="-14.605" y1="1.765" x2="-41.83" y2="-17.62" width="0" layer="19" extent="1-1"/>
+<wire x1="-28.36" y1="29.21" x2="-14.605" y2="1.765" width="0" layer="19" extent="1-1"/>
 </signal>
 <signal name="LEFT_IN_A">
 <contactref element="U$1" pad="1"/>
 <contactref element="U$4" pad="P$5"/>
+<contactref element="R44" pad="2"/>
 <wire x1="-17.145" y1="1.765" x2="-44.29" y2="-11.51" width="0" layer="19" extent="1-1"/>
-</signal>
-<signal name="N$151">
-<contactref element="U$1" pad="4"/>
-</signal>
-<signal name="N$153">
-<contactref element="U$1" pad="2"/>
-</signal>
-<signal name="N$154">
-<contactref element="U$1" pad="8"/>
+<wire x1="-33.44" y1="29.21" x2="-17.145" y2="1.765" width="0" layer="19" extent="1-1"/>
 </signal>
 <signal name="PAIR_LED+">
@@
 </signal>
 <signal name="VCV_M">
+<contactref element="C16" pad="2"/>
+<contactref element="C18" pad="2"/>
 <contactref element="JP9" pad="3"/>
 <contactref element="F1" pad="P$1"/>
 <contactref element="C19" pad="2"/>
+<contactref element="U$1" pad="4"/>
+<contactref element="C27" pad="2"/>
+<contactref element="C28" pad="2"/>
+<contactref element="U$2" pad="4"/>
+<contactref element="U$3" pad="4"/>
+<contactref element="C17" pad="2"/>
 <wire x1="-77.47" y1="-53.34" x2="-101.16" y2="-96.52" width="0" layer="19" extent="1-1"/>
 <wire x1="-42.164" y1="11.43" x2="-77.47" y2="-53.34" width="0" layer="19" extent="1-1"/>
+<wire x1="-23.495" y1="1.765" x2="-42.164" y2="11.43" width="0" layer="19" extent="1-1"/>
+<wire x1="-18.415" y1="1.765" x2="-23.495" y2="1.765" width="0" layer="19" extent="1-1"/>
+<wire x1="-13.335" y1="1.765" x2="-18.415" y2="1.765" width="0" layer="19" extent="1-1"/>
+<wire x1="-14.224" y1="15.24" x2="-13.335" y2="1.765" width="0" layer="19" extent="1-1"/>
+<wire x1="-19.304" y1="15.24" x2="-14.224" y2="15.24" width="0" layer="19" extent="1-1"/>
+<wire x1="-28.36" y1="39.37" x2="-19.304" y2="15.24" width="0" layer="19" extent="1-1"/>
+<wire x1="-33.44" y1="39.37" x2="-28.36" y2="39.37" width="0" layer="19" extent="1-1"/>
+<wire x1="-38.52" y1="39.37" x2="-33.44" y2="39.37" width="0" layer="19" extent="1-1"/>
 </signal>
 <signal name="L_ID">
@@
 <contactref element="JP12" pad="3"/>
 <contactref element="U$4" pad="P$31"/>
+<contactref element="D14" pad="A"/>
 <wire x1="-24.29" y1="-6.27" x2="-77.47" y2="-68.58" width="0" layer="19" extent="1-1"/>
+<wire x1="-38.1" y1="11.43" x2="-24.29" y2="-6.27" width="0" layer="19" extent="1-1"/>
 </signal>
 <signal name="VCC_33">
@@
 <contactref element="C23" pad="2"/>
 <contactref element="C22A" pad="2"/>
-<contactref element="C33" pad="2"/>
 <contactref element="U7" pad="2@1" route="any" routetag="A.VOUT"/>
 <contactref element="U7" pad="2" route="any" routetag="A.VOUT"/>
-<contactref element="L9" pad="2"/>
 <contactref element="Q6" pad="2"/>
 <contactref element="Q14" pad="2"/>
@@
 <contactref element="R30" pad="1"/>
 <contactref element="JP14" pad="5"/>
+<contactref element="C33" pad="2"/>
+<contactref element="L9" pad="2"/>
 <wire x1="-82.55" y1="-83.82" x2="-107.95" y2="-93.04" width="0" layer="19" extent="1-1"/>
 <wire x1="-81.6" y1="-86.36" x2="-82.55" y2="-83.82" width="0" layer="19" extent="1-1"/>
@@
 <wire x1="-16.93" y1="29.21" x2="-42.33" y2="26.67" width="0" layer="19" extent="1-1"/>
 </signal>
-<signal name="D14_A">
-<contactref element="D14" pad="A"/>
-</signal>
 <signal name="OFF">
 <contactref element="R81" pad="2"/>
@@
 <wire x1="-81.6" y1="-91.44" x2="-106.451" y2="-95.961" width="0" layer="19" extent="1-1"/>
 </signal>
+<signal name="RIGHT_IN_A">
+<contactref element="R62" pad="2"/>
+<contactref element="U$2" pad="1"/>
+<wire x1="-43.6" y1="29.21" x2="-22.225" y2="1.765" width="0" layer="19" extent="1-1"/>
+</signal>
+<signal name="RIGHT_IN_B">
+<contactref element="R63" pad="2"/>
+<contactref element="U$2" pad="3"/>
+<wire x1="-38.52" y1="29.21" x2="-19.685" y2="1.765" width="0" layer="19" extent="1-1"/>
+</signal>
 </signals>

Commit message: solved mystery net to motor R, added todos
Connections:
- removed net R26_A: C21.2, R26.1
- removed net R62_B: U$4.P$19
- removed net R63_B: U$4.P$20
- net RIGHT_IN_A: now also U$4.P$19
- net RIGHT_IN_B: now also U$4.P$20
- net VCC_33: now also C21.2, R26.1
Changed lines of the file:
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@@
 </elements>
 <signals>
-<signal name="R62_B">
-<contactref element="U$4" pad="P$19"/>
-</signal>
-<signal name="R63_B">
-<contactref element="U$4" pad="P$20"/>
-</signal>
 <signal name="Q14_B">
 <contactref element="Q14" pad="1"/>
@@
 <contactref element="C33" pad="2"/>
 <contactref element="L9" pad="2"/>
+<contactref element="C21" pad="2"/>
+<contactref element="R26" pad="1"/>
 <wire x1="-82.55" y1="-83.82" x2="-107.95" y2="-93.04" width="0" layer="19" extent="1-1"/>
 <wire x1="-81.6" y1="-86.36" x2="-82.55" y2="-83.82" width="0" layer="19" extent="1-1"/>
@@
 <wire x1="-16.93" y1="24.13" x2="-24.384" y2="15.24" width="0" layer="19" extent="1-1"/>
 <wire x1="-16.93" y1="34.29" x2="-16.93" y2="24.13" width="0" layer="19" extent="1-1"/>
-<wire x1="-16.93" y1="39.37" x2="-16.93" y2="34.29" width="0" layer="19" extent="1-1"/>
-<wire x1="-23.28" y1="36.83" x2="-16.93" y2="34.29" width="0" layer="19" extent="1-1"/>
+<wire x1="-16.93" y1="36.83" x2="-16.93" y2="34.29" width="0" layer="19" extent="1-1"/>
+<wire x1="-16.93" y1="39.37" x2="-16.93" y2="36.83" width="0" layer="19" extent="1-1"/>
+<wire x1="-23.28" y1="36.83" x2="-16.93" y2="36.83" width="0" layer="19" extent="1-1"/>
 <wire x1="-30.9" y1="31.75" x2="-23.28" y2="36.83" width="0" layer="19" extent="1-1"/>
 <wire x1="-32.6" y1="31.75" x2="-30.9" y2="31.75" width="0" layer="19" extent="1-1"/>
 <wire x1="-42.33" y1="21.59" x2="-34.61" y2="10.43" width="0" layer="19" extent="1-1"/>
+<wire x1="-44.03" y1="21.59" x2="-42.33" y2="21.59" width="0" layer="19" extent="1-1"/>
 </signal>
 <signal name="PAIR_BTN">
@@
 <wire x1="-18.63" y1="24.13" x2="-29.63" y2="36.83" width="0" layer="19" extent="1-1"/>
 </signal>
-<signal name="R26_A">
-<contactref element="C21" pad="2"/>
-<contactref element="R26" pad="1"/>
-<wire x1="-16.93" y1="36.83" x2="-44.03" y2="21.59" width="0" layer="19" extent="1-1"/>
-</signal>
 <signal name="BAT+">
 <contactref element="F1" pad="P$2"/>
@@
 <contactref element="R62" pad="2"/>
 <contactref element="U$2" pad="1"/>
+<contactref element="U$4" pad="P$19"/>
+<wire x1="-22.225" y1="1.765" x2="-30.4" y2="-17.62" width="0" layer="19" extent="1-1"/>
 <wire x1="-43.6" y1="29.21" x2="-22.225" y2="1.765" width="0" layer="19" extent="1-1"/>
 </signal>
@@
 <contactref element="R63" pad="2"/>
 <contactref element="U$2" pad="3"/>
+<contactref element="U$4" pad="P$20"/>
+<wire x1="-19.685" y1="1.765" x2="-29.13" y2="-17.62" width="0" layer="19" extent="1-1"/>
 <wire x1="-38.52" y1="29.21" x2="-19.685" y2="1.765" width="0" layer="19" extent="1-1"/>
 </signal>

Commit message: moved parts to new lib
Parts:
- C11, C16, C18, C21, C23, C24, C25, C26, C27, C29, C31, C33, C34, C35, C36, C38, C39, L11, L12, R100, R18, R22, R23, R25, R26, R27, R29, R30, R43, R44, R45, R47_OR_42, R49, R5, R51, R52, R54, R55, R59, R6, R60, R61, R62, R63, R64, R66, R68, R7, R71, R76, R77, R99: device microbuilder:0603-NO -> DROID:0603-NO
- C17, C19, C20A, C22A, C28, R81: device microbuilder:_0805MP -> DROID:_0805MP
- C37: device microbuilder:PANASONIC_D -> DROID:PANASONIC_D
- D14: device microbuilder:SOD-323 -> DROID:SOD-323
- F1: device microbuilder:PTC1812 -> DROID:PTC1812
- JP1, JP2, JP3, JP4, JP5, JP6: device microbuilder:1X02_ROUND -> DROID:1X02_ROUND
- JP10, JP11, JP12: device microbuilder:1X04_ROUND -> DROID:1X04_ROUND
- JP13, JP14: device microbuilder:1X05_ROUND -> DROID:1X05_ROUND
- JP15: device microbuilder:1X06_ROUND -> DROID:1X06_ROUND
- JP7, JP8, JP9: device microbuilder:1X03_ROUND -> DROID:1X03_ROUND
- L13, L14, L9: device microbuilder:0805-NO -> DROID:0805-NO
- Q10, Q13, Q14, Q6: device microbuilder:SOT23-R -> DROID:SOT23-R
- Q11, Q12: device microbuilder:SOT23-WIDE -> DROID:SOT23-WIDE
- U$1, U$2, U$3: device microbuilder:SOIC8_208MIL -> DROID:SOIC8_208MIL
- U$4: device microbuilder:KNRF51822 -> DROID:KNRF51822
- U$5: device microbuilder:GPCD9TP340A -> DROID:GPCD9TP340A
- U7, U8: device microbuilder:SOT89 -> DROID:SOT89

Commit message: major reorganization
Connections:
- net HEAD_OUT_A: now also JP5.2
- net HEAD_OUT_B: no longer JP5.2
- net LEFT_OUT_A: now also JP3.2; no longer JP3.1
- net LEFT_OUT_B: now also JP3.1; no longer JP3.2
- net RIGHT_OUT_A: now also JP4.2; no longer JP4.1
- net RIGHT_OUT_B: now also JP4.1; no longer JP4.2
Changed lines of the file:
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@@
 <signal name="HEAD_OUT_B">
 <contactref element="U$3" pad="5"/>
-<contactref element="JP5" pad="2"/>
 <contactref element="JP5" pad="1"/>
-<wire x1="-73.66" y1="-34.29" x2="-76.2" y2="-34.29" width="0" layer="19" extent="1-1"/>
-<wire x1="-23.495" y1="8.395" x2="-73.66" y2="-34.29" width="0" layer="19" extent="1-1"/>
+<wire x1="-23.495" y1="8.395" x2="-76.2" y2="-34.29" width="0" layer="19" extent="1-1"/>
 </signal>
 <signal name="HEAD_IN_B">
@@
 <signal name="RIGHT_OUT_B">
 <contactref element="U$2" pad="5"/>
-<contactref element="JP4" pad="2"/>
-<wire x1="-18.415" y1="8.395" x2="-67.31" y2="-34.29" width="0" layer="19" extent="1-1"/>
+<contactref element="JP4" pad="1"/>
+<wire x1="-18.415" y1="8.395" x2="-69.85" y2="-34.29" width="0" layer="19" extent="1-1"/>
 </signal>
 <signal name="RIGHT_OUT_A">
 <contactref element="U$2" pad="7"/>
-<contactref element="JP4" pad="1"/>
-<wire x1="-20.955" y1="8.395" x2="-69.85" y2="-34.29" width="0" layer="19" extent="1-1"/>
+<contactref element="JP4" pad="2"/>
+<wire x1="-20.955" y1="8.395" x2="-67.31" y2="-34.29" width="0" layer="19" extent="1-1"/>
 </signal>
 <signal name="LEFT_OUT_B">
 <contactref element="U$1" pad="5"/>
-<contactref element="JP3" pad="2"/>
-<wire x1="-13.335" y1="8.395" x2="-60.96" y2="-34.29" width="0" layer="19" extent="1-1"/>
+<contactref element="JP3" pad="1"/>
+<wire x1="-13.335" y1="8.395" x2="-63.5" y2="-34.29" width="0" layer="19" extent="1-1"/>
 </signal>
 <signal name="LEFT_OUT_A">
 <contactref element="U$1" pad="7"/>
-<contactref element="JP3" pad="1"/>
-<wire x1="-15.875" y1="8.395" x2="-63.5" y2="-34.29" width="0" layer="19" extent="1-1"/>
+<contactref element="JP3" pad="2"/>
+<wire x1="-15.875" y1="8.395" x2="-60.96" y2="-34.29" width="0" layer="19" extent="1-1"/>
 </signal>
 <signal name="LEFT_IN_B">
@@
 <contactref element="U$4" pad="P$9"/>
 <contactref element="R5" pad="1"/>
-<contactref element="U$1" pad="6"/>
-<contactref element="U$2" pad="6"/>
 <contactref element="U$3" pad="6"/>
 <contactref element="C38" pad="1"/>
@@
 <contactref element="Q12" pad="2"/>
 <contactref element="R61" pad="2"/>
-<contactref element="C26" pad="2"/>
 <contactref element="R66" pad="1"/>
 <contactref element="C31" pad="1"/>
@@
 <contactref element="C18" pad="1"/>
 <contactref element="C19" pad="1"/>
-<contactref element="C34" pad="1"/>
 <contactref element="C24" pad="1"/>
 <contactref element="C25" pad="1"/>
@@
 <contactref element="C39" pad="1"/>
 <contactref element="L14" pad="1"/>
+<contactref element="U$1" pad="6"/>
+<contactref element="U$2" pad="6"/>
+<contactref element="C34" pad="1"/>
+<contactref element="C26" pad="2"/>
 <wire x1="-92.824" y1="-95.25" x2="-114.071" y2="-95.961" width="0" layer="19" extent="1-1"/>
 <wire x1="-83.5" y1="-91.44" x2="-92.824" y2="-95.25" width="0" layer="19" extent="1-1"/>
@@
 <contactref element="U$5" pad="23"/>
 <contactref element="U$5" pad="32"/>
-<contactref element="C23" pad="2"/>
 <contactref element="C22A" pad="2"/>
 <contactref element="U7" pad="2@1" route="any" routetag="A.VOUT"/>
@@
 <contactref element="C21" pad="2"/>
 <contactref element="R26" pad="1"/>
+<contactref element="C23" pad="2"/>
 <wire x1="-82.55" y1="-83.82" x2="-107.95" y2="-93.04" width="0" layer="19" extent="1-1"/>
 <wire x1="-81.6" y1="-86.36" x2="-82.55" y2="-83.82" width="0" layer="19" extent="1-1"/>
@@
 <signal name="HEAD_OUT_A">
 <contactref element="U$3" pad="7"/>
+<contactref element="JP5" pad="2"/>
+<wire x1="-26.035" y1="8.395" x2="-73.66" y2="-34.29" width="0" layer="19" extent="1-1"/>
 </signal>
 <signal name="R61_A">
