File: DROID.brd (EAGLE design)
At the start: 160 x 100 mm, 92 parts

Commit message: more organization
Parts:
- removed R26, R30, R76, R77: 0, DROID:0603-NO
Connections:
- net P0.14 renamed MM_RESET_OUT
- net Q12_C renamed MM_RESET
- net U7_VIN renamed 9V_IN
- removed net R76_A: C11.2, R76.1
- removed net U8_VOUT: C24.2, C25.2, C36.2, R25.1, R77.1, R77.2, U8.2, U8.2@1
- new net 3.3V: C24.2, C25.2, C36.2, R25.1, U8.2, U8.2@1
- new net 5V: C20A.2, C21.2, C22A.2, C23.2, C33.2, L9.2, Q13.2, Q14.2, Q6.2, U7.2, U7.2@1
- net VCC_33: now also C11.2; no longer C20A.2, C21.2, C22A.2, C23.2, C33.2, JP14.5, L9.2, Q13.2, Q14.2, Q6.2, R26.1, R26.2, R30.1, R30.2, R76.2, U7.2, U7.2@1
Changed lines of the file:
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@@
 <attribute name="VALUE" x="-35.052" y="20.828" size="0.4064" layer="27" font="vector" ratio="10"/>
-</element>
-<element name="R26" library="DROID" package="0603-NO" value="0" x="-43.18" y="21.59" smashed="yes">
-<attribute name="NAME" x="-41.402" y="21.463" size="0.8128" layer="25" font="vector" ratio="18"/>
-<attribute name="VALUE" x="-41.402" y="20.828" size="0.4064" layer="27" font="vector" ratio="10"/>
-</element>
-<element name="R76" library="DROID" package="0603-NO" value="0" x="-17.78" y="24.13" smashed="yes">
-<attribute name="NAME" x="-16.002" y="24.003" size="0.8128" layer="25" font="vector" ratio="18"/>
-<attribute name="VALUE" x="-16.002" y="23.368" size="0.4064" layer="27" font="vector" ratio="10"/>
 </element>
 <element name="R59" library="DROID" package="0603-NO" value="300K" x="-24.13" y="24.13" smashed="yes">
@@
 <attribute name="NAME" x="-19.812" y="31.623" size="0.8128" layer="25" font="vector" ratio="18"/>
 <attribute name="VALUE" x="-19.812" y="30.988" size="0.4064" layer="27" font="vector" ratio="10"/>
-</element>
-<element name="R77" library="DROID" package="0603-NO" value="0" x="-26.67" y="31.75" smashed="yes">
-<attribute name="NAME" x="-24.892" y="31.623" size="0.8128" layer="25" font="vector" ratio="18"/>
-<attribute name="VALUE" x="-24.892" y="30.988" size="0.4064" layer="27" font="vector" ratio="10"/>
-</element>
-<element name="R30" library="DROID" package="0603-NO" value="0" x="-31.75" y="31.75" smashed="yes">
-<attribute name="NAME" x="-29.972" y="31.623" size="0.8128" layer="25" font="vector" ratio="18"/>
-<attribute name="VALUE" x="-29.972" y="30.988" size="0.4064" layer="27" font="vector" ratio="10"/>
 </element>
 <element name="R54" library="DROID" package="0603-NO" value="100" x="-36.83" y="31.75" smashed="yes">
@@
 <wire x1="-23.28" y1="24.13" x2="-16.51" y2="12.43" width="0" layer="19" extent="1-1"/>
 </signal>
-<signal name="U8_VOUT">
-<contactref element="R77" pad="1"/>
+<signal name="3.3V">
 <contactref element="C25" pad="2"/>
 <contactref element="C24" pad="2"/>
 <contactref element="R25" pad="1"/>
-<contactref element="R77" pad="2"/>
 <contactref element="C36" pad="2"/>
 <contactref element="U8" pad="2@1" route="any" routetag="A.VOUT"/>
 <contactref element="U8" pad="2" route="any" routetag="A.VOUT"/>
 <wire x1="-24.98" y1="21.59" x2="-115.57" y2="-93.04" width="0" layer="19" extent="1-1"/>
-<wire x1="-25.82" y1="31.75" x2="-24.98" y2="21.59" width="0" layer="19" extent="1-1"/>
-<wire x1="-27.52" y1="31.75" x2="-25.82" y2="31.75" width="0" layer="19" extent="1-1"/>
-<wire x1="-29.63" y1="34.29" x2="-27.52" y2="31.75" width="0" layer="19" extent="1-1"/>
+<wire x1="-29.63" y1="34.29" x2="-24.98" y2="21.59" width="0" layer="19" extent="1-1"/>
 <wire x1="-35.98" y1="34.29" x2="-29.63" y2="34.29" width="0" layer="19" extent="1-1"/>
 <wire x1="-43.6" y1="39.37" x2="-35.98" y2="34.29" width="0" layer="19" extent="1-1"/>
@@
 <wire x1="-37.68" y1="21.59" x2="-37.78" y2="1.54" width="0" layer="19" extent="1-1"/>
 </signal>
-<signal name="Q12_C">
+<signal name="MM_RESET">
 <contactref element="C29" pad="2"/>
 <contactref element="Q12" pad="3"/>
@@
 <wire x1="-26.59" y1="-17.62" x2="-77.47" y2="-63.5" width="0" layer="19" extent="1-1"/>
 </signal>
-<signal name="P0.14">
+<signal name="MM_RESET_OUT">
 <contactref element="U$4" pad="P$25"/>
+<contactref element="R71" pad="2"/>
 <contactref element="R68" pad="2"/>
-<contactref element="R71" pad="2"/>
 <wire x1="-29.63" y1="21.59" x2="-24.29" y2="-13.89" width="0" layer="19" extent="1-1"/>
 <wire x1="-35.98" y1="21.59" x2="-29.63" y2="21.59" width="0" layer="19" extent="1-1"/>
@@
 <contactref element="JP12" pad="4"/>
 <contactref element="JP15" pad="1"/>
-<contactref element="U$4" pad="P$8"/>
-<contactref element="R76" pad="2"/>
-<contactref element="C31" pad="2"/>
 <contactref element="U$5" pad="2"/>
 <contactref element="U$5" pad="4"/>
@@
 <contactref element="U$5" pad="23"/>
 <contactref element="U$5" pad="32"/>
-<contactref element="C22A" pad="2"/>
-<contactref element="U7" pad="2@1" route="any" routetag="A.VOUT"/>
-<contactref element="U7" pad="2" route="any" routetag="A.VOUT"/>
-<contactref element="Q6" pad="2"/>
-<contactref element="Q14" pad="2"/>
-<contactref element="Q13" pad="2"/>
-<contactref element="C20A" pad="2"/>
-<contactref element="R26" pad="2"/>
-<contactref element="R30" pad="2"/>
-<contactref element="R30" pad="1"/>
-<contactref element="JP14" pad="5"/>
-<contactref element="C33" pad="2"/>
-<contactref element="L9" pad="2"/>
-<contactref element="C21" pad="2"/>
-<contactref element="R26" pad="1"/>
-<contactref element="C23" pad="2"/>
-<wire x1="-82.55" y1="-83.82" x2="-107.95" y2="-93.04" width="0" layer="19" extent="1-1"/>
-<wire x1="-81.6" y1="-86.36" x2="-82.55" y2="-83.82" width="0" layer="19" extent="1-1"/>
-<wire x1="-72.39" y1="-78.74" x2="-82.55" y2="-83.82" width="0" layer="19" extent="1-1"/>
-<wire x1="-74.93" y1="-68.58" x2="-72.39" y2="-78.74" width="0" layer="19" extent="1-1"/>
+<contactref element="C11" pad="2"/>
+<contactref element="U$4" pad="P$8"/>
+<contactref element="C31" pad="2"/>
+<wire x1="-74.93" y1="-68.58" x2="-82.55" y2="-83.82" width="0" layer="19" extent="1-1"/>
 <wire x1="-36.72" y1="-38.32" x2="-74.93" y2="-68.58" width="0" layer="19" extent="1-1"/>
 <wire x1="-27.72" y1="-38.32" x2="-36.72" y2="-38.32" width="0" layer="19" extent="1-1"/>
@@
 <wire x1="-31.72" y1="-20.32" x2="-28.72" y2="-20.32" width="0" layer="19" extent="1-1"/>
 <wire x1="-44.29" y1="-15.32" x2="-31.72" y2="-20.32" width="0" layer="19" extent="1-1"/>
-<wire x1="-34.61" y1="10.43" x2="-44.29" y2="-15.32" width="0" layer="19" extent="1-1"/>
-<wire x1="-28.26" y1="10.43" x2="-34.61" y2="10.43" width="0" layer="19" extent="1-1"/>
-<wire x1="-29.464" y1="15.24" x2="-28.26" y2="10.43" width="0" layer="19" extent="1-1"/>
-<wire x1="-24.384" y1="15.24" x2="-29.464" y2="15.24" width="0" layer="19" extent="1-1"/>
-<wire x1="-21.91" y1="10.43" x2="-24.384" y2="15.24" width="0" layer="19" extent="1-1"/>
-<wire x1="-16.93" y1="24.13" x2="-24.384" y2="15.24" width="0" layer="19" extent="1-1"/>
-<wire x1="-16.93" y1="34.29" x2="-16.93" y2="24.13" width="0" layer="19" extent="1-1"/>
-<wire x1="-16.93" y1="36.83" x2="-16.93" y2="34.29" width="0" layer="19" extent="1-1"/>
-<wire x1="-16.93" y1="39.37" x2="-16.93" y2="36.83" width="0" layer="19" extent="1-1"/>
-<wire x1="-23.28" y1="36.83" x2="-16.93" y2="36.83" width="0" layer="19" extent="1-1"/>
-<wire x1="-30.9" y1="31.75" x2="-23.28" y2="36.83" width="0" layer="19" extent="1-1"/>
-<wire x1="-32.6" y1="31.75" x2="-30.9" y2="31.75" width="0" layer="19" extent="1-1"/>
-<wire x1="-42.33" y1="21.59" x2="-34.61" y2="10.43" width="0" layer="19" extent="1-1"/>
-<wire x1="-44.03" y1="21.59" x2="-42.33" y2="21.59" width="0" layer="19" extent="1-1"/>
+<wire x1="-29.63" y1="36.83" x2="-44.29" y2="-15.32" width="0" layer="19" extent="1-1"/>
+<wire x1="-16.93" y1="39.37" x2="-29.63" y2="36.83" width="0" layer="19" extent="1-1"/>
 </signal>
 <signal name="PAIR_BTN">
@@
 <wire x1="-29.464" y1="2.54" x2="-82.55" y2="-53.34" width="0" layer="19" extent="1-1"/>
 </signal>
-<signal name="U7_VIN">
+<signal name="9V_IN">
 <contactref element="R54" pad="1"/>
 <contactref element="Q10" pad="2"/>
@@
 <wire x1="-18.63" y1="29.21" x2="-44.13" y2="1.54" width="0" layer="19" extent="1-1"/>
 </signal>
-<signal name="R76_A">
-<contactref element="C11" pad="2"/>
-<contactref element="R76" pad="1"/>
-<wire x1="-18.63" y1="24.13" x2="-29.63" y2="36.83" width="0" layer="19" extent="1-1"/>
-</signal>
 <signal name="BAT+">
 <contactref element="F1" pad="P$2"/>
@@
 <wire x1="-38.52" y1="29.21" x2="-19.685" y2="1.765" width="0" layer="19" extent="1-1"/>
 </signal>
+<signal name="5V">
+<contactref element="C22A" pad="2"/>
+<contactref element="U7" pad="2@1" route="any" routetag="A.VOUT"/>
+<contactref element="U7" pad="2" route="any" routetag="A.VOUT"/>
+<contactref element="Q6" pad="2"/>
+<contactref element="Q14" pad="2"/>
+<contactref element="Q13" pad="2"/>
+<contactref element="C20A" pad="2"/>
+<contactref element="C33" pad="2"/>
+<contactref element="L9" pad="2"/>
+<contactref element="C21" pad="2"/>
+<contactref element="C23" pad="2"/>
+<wire x1="-81.6" y1="-86.36" x2="-107.95" y2="-93.04" width="0" layer="19" extent="1-1"/>
+<wire x1="-34.61" y1="10.43" x2="-81.6" y2="-86.36" width="0" layer="19" extent="1-1"/>
+<wire x1="-28.26" y1="10.43" x2="-34.61" y2="10.43" width="0" layer="19" extent="1-1"/>
+<wire x1="-29.464" y1="15.24" x2="-28.26" y2="10.43" width="0" layer="19" extent="1-1"/>
+<wire x1="-24.384" y1="15.24" x2="-29.464" y2="15.24" width="0" layer="19" extent="1-1"/>
+<wire x1="-21.91" y1="10.43" x2="-24.384" y2="15.24" width="0" layer="19" extent="1-1"/>
+<wire x1="-16.93" y1="34.29" x2="-24.384" y2="15.24" width="0" layer="19" extent="1-1"/>
+<wire x1="-16.93" y1="36.83" x2="-16.93" y2="34.29" width="0" layer="19" extent="1-1"/>
+<wire x1="-23.28" y1="36.83" x2="-16.93" y2="36.83" width="0" layer="19" extent="1-1"/>
+</signal>
 </signals>
