File: DROID.sch (EAGLE design)
At the start: 92 parts

Commit message: saving before cleanup
Connections:
- removed net C16_B: C16.2
- removed net C17_B: C17.2
- removed net C18_B: C18.2
- removed net C27_B: C27.2
- removed net C28_B: C28.2
- removed net D14_A: D14.A
- removed net N$135: U$3.VCC
- removed net N$137: U$3.NC
- removed net N$138: U$3.NC@1
- removed net N$143: U$2.VCC
- removed net N$145: U$2.NC
- removed net N$146: U$2.NC@1
- removed net N$151: U$1.VCC
- removed net N$153: U$1.NC
- removed net N$154: U$1.NC@1
- removed net N$16: R47_OR_42.2
- removed net R43_B: R43.2
- removed net R44_B: R44.2
- removed net R45_B: R45.2
- net HEAD_IN_A: now also R43.2
- net HEAD_IN_B: now also R45.2
- net LEFT_IN_A: now also R44.2
- net LEFT_IN_B: now also R47_OR_42.2
- net R62_B: no longer R62.2
- net R63_B: no longer R63.2
- net RIGHT_IN_A: now also R62.2
- net RIGHT_IN_B: now also R63.2
- net SWDIO: now also D14.A
- net VCV_M: now also C16.2, C17.2, C18.2, C27.2, C28.2, U$1.VCC, U$2.VCC, U$3.VCC
Other:
- note removed: "Connections to passives have the _B net towards the nrf or mystery module"
- moved on the sheet: C16, C17, C18, C19, C24, C25, C27, C28, C33, C34, C35, C36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

Commit message: solved mystery net to motor R, added todos
Connections:
- removed net R26_A: C21.2, R26.1
- removed net R62_B: U$4.P0.8
- removed net R63_B: U$4.P0.9
- net RIGHT_IN_A: now also U$4.P0.8
- net RIGHT_IN_B: now also U$4.P0.9
- net VCC_33: now also C21.2, R26.1
Other:
- note added: "TODO: * More cleanup * Change H-Bridge Symbol to have out on the other side and pins closer to real life * Check actual voltages * Try to identify voltage dividers * Re-Check SWDIO to Diode * Summarize Connections to NRF and Mystery Module"
- moved on the sheet: C20A, C21, C22A, C23, C26, C29, C35, JP11, JP12, JP15, L9, Q11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

Commit message: adding library export
Other:
- note added: "Mystery Module"
- note added: "Totally not an NRF51822"
- moved on the sheet: C29, JP11, JP12, Q12, R5, R68, R71

Commit message: moved parts to new lib
Parts:
- C11, C16, C18, C21, C23, C24, C25, C26, C27, C29, C31, C33, C34, C35, C36, C38, C39: device microbuilder:CAP_CERAMIC0603_NO -> DROID:CAP_CERAMIC0603_NO
- C17, C19, C20A, C22A, C28: device microbuilder:CAP_CERAMIC_0805MP -> DROID:CAP_CERAMIC_0805MP
- C37: device microbuilder:CAP_ELECTROLYTICPANASONIC_D -> DROID:CAP_ELECTROLYTICPANASONIC_D
- D14: device microbuilder:DIODESOD-323 -> DROID:DIODESOD-323
- F1: device microbuilder:PTC1812 -> DROID:PTC1812
- JP1, JP2, JP3, JP4, JP5, JP6: device microbuilder:HEADER-1X2ROUND -> DROID:HEADER-1X2ROUND
- JP10, JP11, JP12: device microbuilder:HEADER-1X4ROUND -> DROID:HEADER-1X4ROUND
- JP13, JP14: device microbuilder:HEADER-1X5ROUND -> DROID:HEADER-1X5ROUND
- JP15: device microbuilder:HEADER-1X6ROUND -> DROID:HEADER-1X6ROUND
- JP7, JP8, JP9: device microbuilder:HEADER-1X3ROUND -> DROID:HEADER-1X3ROUND
- L11, L12: device microbuilder:INDUCTOR0603_NO -> DROID:INDUCTOR0603_NO
- L13, L14, L9: device microbuilder:INDUCTOR0805-NO -> DROID:INDUCTOR0805-NO
- Q10, Q13, Q14, Q6: device microbuilder:TRANSISTOR_PNPSOT23-REFLOW -> DROID:TRANSISTOR_PNPSOT23-REFLOW
- Q11, Q12: device microbuilder:TRANSISTOR_NPNWIDE -> DROID:TRANSISTOR_NPNWIDE
- R100, R18, R22, R23, R25, R26, R27, R29, R30, R43, R44, R45, R47_OR_42, R49, R5, R51, R52, R54, R55, R59, R6, R60, R61, R62, R63, R64, R66, R68, R7, R71, R76, R77, R99: device microbuilder:RESISTOR_0603_NOOUT -> DROID:RESISTOR_0603_NOOUT
- R81: device microbuilder:RESISTOR_0805MP -> DROID:RESISTOR_0805MP
- U$1, U$2, U$3: device microbuilder:AM1037A -> DROID:AM1037A
- U$4: device microbuilder:KNRF51822_A24 -> DROID:KNRF51822_A24
- U$5: device microbuilder:GPCD9TP340A_DROID -> DROID:GPCD9TP340A_DROID
- U7, U8: device microbuilder:ME62XX -> DROID:ME62XX

Commit message: major reorganization
Connections:
- net HEAD_OUT_A: now also JP5.2
- net HEAD_OUT_B: no longer JP5.2
- net LEFT_OUT_A: now also JP3.2; no longer JP3.1
- net LEFT_OUT_B: now also JP3.1; no longer JP3.2
- net RIGHT_OUT_A: now also JP4.2; no longer JP4.1
- net RIGHT_OUT_B: now also JP4.1; no longer JP4.2
Other:
- note removed: "RIGHT"
- moved on the sheet: C11, C20A, C21, C22A, C23, C26, C27, C28, C29, C31, C33, C34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

Commit message: more organization
Parts:
- removed R26, R30, R76, R77: 0, DROID:RESISTOR_0603_NOOUT
Connections:
- net P0.14 renamed MM_RESET_OUT
- net Q12_C renamed MM_RESET
- net U7_VIN renamed 9V_IN
- removed net R76_A: C11.2, R76.1
- removed net U8_VOUT: C24.2, C25.2, C36.2, R25.1, R77.1, R77.2, U8.VOUT
- new net 3.3V: C24.2, C25.2, C36.2, R25.1, U8.VOUT
- new net 5V: C20A.2, C21.2, C22A.2, C23.2, C33.2, L9.2, Q13.E, Q14.E, Q6.E, U7.VOUT
- net VCC_33: now also C11.2; no longer C20A.2, C21.2, C22A.2, C23.2, C33.2, JP14.5, L9.2, Q13.E, Q14.E, Q6.E, R26.1, R26.2, R30.1, R30.2, R76.2, U7.VOUT
Other:
- note added: "EXT_FLASH_SPI"
- note added: "HEAD RGB LED"
- note added: "L & R LEG LEDS"
- note added: "ONE TIME PROGRAMMING I2C PORT"
- note added: "SPEAKER OUT"
- note added: "TODO: * More cleanup * Check actual voltages * Try to identify voltage dividers * Re-Check SWDIO to Diode * Summarize Connections to NRF and Mystery Module"
- note removed: "TODO: * More cleanup * Change H-Bridge Symbol to have out on the other side and pins closer to real life * Check actual voltages * Try to identify voltage dividers * Re-Check SWDIO to Diode * Summarize Connections to NRF and Mystery Module"
- moved on the sheet: C16, C17, C18, C19, C20A, C21, C22A, C23, C24, C25, C26, C27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
